File: 0.0.1-custom-pcb/chocPcb/AdafruitNeoKeyChocSocketBreakout.kicad_pcb (KiCad board)
At the start: 2 copper layers, 19.2 x 24.1 mm, 39 parts, among them SW1 MX SOCKET

Commit message: add 3d models to choc pcb
Parts:
- LED1, SW1: moved to F.Cu
