File: 0.0.1-custom-pcb/columnBreakout/columnBreakout.kicad_sch (KiCad schematic)
At the start: 7 parts, among them J1 HC-FPC-0.5-12P-FH20, J2 HC-FPC-0.5-6P-FH20, J3 HC-FPC-0.5-6P-FH20, J4 HC-FPC-0.5-6P-FH20, J5 HC-FPC-0.5-6P-FH20, J6 HC-FPC-0.5-6P-FH20, J7 HC-FPC-0.5-6P-FH20

Commit message: made order for 100 chocPcb and 5 columnBreakout
Other:
- title: (none) -> columnBreakout
Changed lines of the file:
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@@
 (generator_version "9.0")
 (paper "A4")
+(title_block
+  (title "columnBreakout")
+  (rev "1")
+)
 (no_connect (at 237.49 60.96)
 )
