File: 0.0.1-custom-pcb/rightPinkieBreakout/columnBreakout.kicad_pcb (KiCad board)
At the start: 2 copper layers, 28.7 x 63.3 mm, 17 parts, among them J1 HC-FPC-0.5-12P-FH20, J10 HC-FPC-0.5-6P-FH20, J11 HC-FPC-0.5-6P-FH20, J12 HC-FPC-0.5-6P-FH20, J13 HC-FPC-0.5-6P-FH20, J2 HC-FPC-0.5-6P-FH20, J3 HC-FPC-0.5-6P-FH20, J4 HC-FPC-0.5-6P-FH20, J5 HC-FPC-0.5-6P-FH20, J6 HC-FPC-0.5-6P-FH20, J7 HC-FPC-0.5-6P-FH20, J8 HC-FPC-0.5-6P-FH20, J9 HC-FPC-0.5-6P-FH20

Commit message: right pinkie breakout rev1 is ready for fab/assembly
Parts:
- renumbered J11 to J10, J10 to J11, J9 to J12, J8 to J13, J13 to J8, J12 to J9
Connections:
- J10 pad 6: /C5 -> /C6
- J11 pad 6: /C5 -> /C6
- J12 pad 6: /C5 -> /C6
- J13 pad 6: /C5 -> /C6
- J2 pad 6: /C6 -> /C5
- J3 pad 6: /C6 -> /C5
- J4 pad 6: /C6 -> /C5
- J5 pad 6: /C6 -> /C5
- J6 pad 6: /C6 -> /C5
- J7 pad 6: /C6 -> /C5
- J8 pad 6: /C5 -> /C6
- J9 pad 6: /C5 -> /C6
Routing:
- net /C6: track 55.4 -> 65.2 mm
- net /C5: track 63.8 -> 55.3 mm
- net /IN34: track 60.9 -> 54.3 mm
