File: 0.0.1-custom-pcb/rightPinkieBreakout/columnBreakout.kicad_sch (KiCad schematic)
At the start: 13 parts, among them J1 HC-FPC-0.5-12P-FH20, J10 HC-FPC-0.5-6P-FH20, J11 HC-FPC-0.5-6P-FH20, J12 HC-FPC-0.5-6P-FH20, J13 HC-FPC-0.5-6P-FH20, J2 HC-FPC-0.5-6P-FH20, J3 HC-FPC-0.5-6P-FH20, J4 HC-FPC-0.5-6P-FH20, J5 HC-FPC-0.5-6P-FH20, J6 HC-FPC-0.5-6P-FH20, J7 HC-FPC-0.5-6P-FH20, J8 HC-FPC-0.5-6P-FH20, J9 HC-FPC-0.5-6P-FH20

Commit message: right pinkie breakout rev1 is ready for fab/assembly
Parts:
- renumbered J11 to J10, J10 to J11, J9 to J12, J8 to J13, J13 to J8, J12 to J9
Connections:
- net C5: now also J2.6, J3.6, J4.6, J5.6, J6.6, J7.6; no longer J10.6, J11.6, J12.6, J13.6, J8.6, J9.6
- net C6: now also J10.6, J11.6, J12.6, J13.6, J8.6, J9.6; no longer J2.6, J3.6, J4.6, J5.6, J6.6, J7.6
Changed lines of the file:
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@@
 		)
 	)
-	(label "C6"
+	(label "C5"
 		(at 97.79 46.99 180)
 		(effects
@@
 		)
 	)
-	(label "C6"
+	(label "C5"
 		(at 130.81 45.72 180)
 		(effects
@@
 		)
 	)
-	(label "C6"
+	(label "C5"
 		(at 161.29 45.72 180)
 		(effects
@@
 		)
 	)
-	(label "C6"
+	(label "C5"
 		(at 190.5 45.72 180)
 		(effects
@@
 		)
 	)
-	(label "C6"
+	(label "C5"
 		(at 224.79 44.45 180)
 		(effects
@@
 		)
 	)
-	(label "C6"
+	(label "C5"
 		(at 256.54 44.45 180)
 		(effects
@@
 		)
 	)
-	(label "C5"
+	(label "C6"
 		(at 163.83 87.63 180)
 		(effects
@@
 		)
 	)
-	(label "C5"
+	(label "C6"
 		(at 227.33 86.36 180)
 		(effects
@@
 		)
 	)
-	(label "C5"
+	(label "C6"
 		(at 133.35 87.63 180)
 		(effects
@@
 		)
 	)
-	(label "C5"
+	(label "C6"
 		(at 193.04 87.63 180)
 		(effects
@@
 		)
 	)
-	(label "C5"
+	(label "C6"
 		(at 259.08 86.36 180)
 		(effects
@@
 		)
 	)
-	(label "C5"
+	(label "C6"
 		(at 100.33 88.9 180)
 		(effects
@@
 		(on_board yes)
 		(dnp no)
-		(property "Reference" "J8"
+		(property "Reference" "J13"
 			(at 103.124 62.992 0)
 			(effects
@@
 			(project "columnBreakout"
 				(path "/b2acabc5-938f-4880-a5a5-3139adf73df1"
-					(reference "J8")
+					(reference "J13")
 					(unit 1)
 				)
@@
 		(on_board yes)
 		(dnp no)
-		(property "Reference" "J11"
+		(property "Reference" "J10"
 			(at 196.596 61.976 0)
 			(effects
@@
 			(project "columnBreakout"
 				(path "/b2acabc5-938f-4880-a5a5-3139adf73df1"
-					(reference "J11")
+					(reference "J10")
 					(unit 1)
 				)
@@
 		(on_board yes)
 		(dnp no)
-		(property "Reference" "J9"
+		(property "Reference" "J12"
 			(at 137.16 63.246 0)
 			(effects
@@
 			(project "columnBreakout"
 				(path "/b2acabc5-938f-4880-a5a5-3139adf73df1"
-					(reference "J9")
+					(reference "J12")
 					(unit 1)
 				)
@@
 		(on_board yes)
 		(dnp no)
-		(property "Reference" "J10"
+		(property "Reference" "J11"
 			(at 167.386 61.976 0)
 			(effects
@@
 			(project "columnBreakout"
 				(path "/b2acabc5-938f-4880-a5a5-3139adf73df1"
-					(reference "J10")
+					(reference "J11")
 					(unit 1)
 				)
@@
 		(on_board yes)
 		(dnp no)
-		(property "Reference" "J13"
+		(property "Reference" "J8"
 			(at 262.636 62.738 0)
 			(effects
@@
 			(project "columnBreakout"
 				(path "/b2acabc5-938f-4880-a5a5-3139adf73df1"
-					(reference "J13")
+					(reference "J8")
 					(unit 1)
 				)
@@
 		(on_board yes)
 		(dnp no)
-		(property "Reference" "J12"
+		(property "Reference" "J9"
 			(at 231.648 62.738 0)
 			(effects
@@
 			(project "columnBreakout"
 				(path "/b2acabc5-938f-4880-a5a5-3139adf73df1"
-					(reference "J12")
+					(reference "J9")
 					(unit 1)
 				)
