File: 0.0.1-custom-pcb/rightPointerThumbBreakout/columnBreakout.kicad_sch (KiCad schematic)
At the start: 17 parts, among them J1 HC-FPC-0.5-12P-FH20, J10 HC-FPC-0.5-6P-FH20, J11 HC-FPC-0.5-6P-FH20, J12 HC-FPC-0.5-6P-FH20, J13 HC-FPC-0.5-6P-FH20, J14 HC-FPC-0.5-6P-FH20, J15 HC-FPC-0.5-6P-FH20, J16 HC-FPC-0.5-6P-FH20, J17 HC-FPC-0.5-6P-FH20, J2 HC-FPC-0.5-6P-FH20, J3 HC-FPC-0.5-6P-FH20, J4 HC-FPC-0.5-6P-FH20, J5 HC-FPC-0.5-6P-FH20, J6 HC-FPC-0.5-6P-FH20, J7 HC-FPC-0.5-6P-FH20, J8 HC-FPC-0.5-6P-FH20, J9 HC-FPC-0.5-6P-FH20

Commit message: right pointerThumb before review
Parts:
- J1: value HC-FPC-0.5-12P-FH20 -> HC-FPC-0.5-14P-FH20; footprint EasyEDA:FPC-SMD_12P-P0.50_HC-FPC-0.5-12P-FH20 -> EasyEDA:FPC-SMD_14P-P0.50_HC-FPC-0.5-14P-FH20; symbol EasyEDA:HC-FPC-0.5-12P-FH20 -> EasyEDA:HC-FPC-0.5-14P-FH20; LCSC Part C19273928 -> C19273929; MPN HC-FPC-0.5-12P-FH20 -> HC-FPC-0.5-14P-FH20
Connections:
- net C0: now also J1.13
- net R0: now also J12.1; no longer J17.1, J8.1
- net R1: now also J13.1, J8.1; no longer J16.1, J9.1
- net R2: now also J17.1, J9.1; no longer J10.1, J15.1
- net R3: now also J10.1, J16.1; no longer J11.1, J14.1
- net R4: now also J11.1, J15.1; no longer J12.1
- net R5: now also J14.1; no longer J13.1
- net IN28 renamed IN0
- net IN29 renamed IN1
- net IN30 renamed IN2
- net IN31 renamed IN3
- net IN32 renamed IN4
- net IN33 renamed IN5
- net IN34 renamed IN6
- net IN6: no longer J17.5
- net IN35 renamed IN13
- net IN13: no longer J8.4, J9.5
- net IN36 renamed IN14
- net IN14: no longer J10.5, J9.4
- net IN37 renamed IN15
- net IN15: no longer J10.4, J11.5
- net IN38 renamed IN10
- net IN10: no longer J14.4
- net IN39 renamed IN11
- net IN40 renamed IN12
- net IN12: now also J17.5; no longer J1.9
- new net IN16: J1.9, J14.4
- new net IN7: J8.4, J9.5
- new net IN8: J10.5, J9.4
- new net IN9: J10.4, J11.5
Other:
- title: columnBreakout -> rightPointerThumbBreakout
Changed lines of the file:
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@@
 	(paper "A4")
 	(title_block
-		(title "columnBreakout")
+		(title "rightPointerThumbBreakout")
 		(rev "1")
 	)
 	(no_connect
-		(at 38.1 135.89)
-	)
-	(no_connect
 		(at 48.26 102.87)
 	)
 	(no_connect
-		(at 48.26 140.97)
+		(at 48.26 146.05)
 	)
 	(no_connect
@@
 	)
 	(no_connect
+		(at 38.1 140.97)
+	)
+	(no_connect
 		(at 232.41 110.49)
 	)
@@
 		(at 167.64 68.58)
 	)
-	(label "IN35"
+	(wire
+		(pts
+			(xy 35.56 138.43) (xy 38.1 138.43)
+		)
+		(stroke
+			(width 0)
+			(type default)
+		)
+	)
+	(label "IN7"
 		(at 194.31 82.55 180)
 		(effects
@@
 		)
 	)
-	(label "R5"
+	(label "R1"
 		(at 226.06 115.57 180)
 		(effects
@@
 		)
 	)
-	(label "IN40"
+	(label "IN16"
 		(at 38.1 128.27 180)
 		(effects
@@
 		)
 	)
-	(label "IN28"
+	(label "IN0"
 		(at 38.1 130.81 180)
 		(effects
@@
 		)
 	)
-	(label "IN33"
+	(label "IN5"
 		(at 97.79 44.45 180)
 		(effects
@@
 		)
 	)
-	(label "IN34"
+	(label "IN6"
 		(at 97.79 41.91 180)
 		(effects
@@
 		)
 	)
-	(label "IN32"
+	(label "IN4"
 		(at 130.81 43.18 180)
 		(effects
@@
 		)
 	)
-	(label "IN33"
+	(label "IN5"
 		(at 130.81 40.64 180)
 		(effects
@@
 		)
 	)
-	(label "IN31"
+	(label "IN3"
 		(at 161.29 43.18 180)
 		(effects
@@
 		)
 	)
-	(label "IN32"
+	(label "IN4"
 		(at 161.29 40.64 180)
 		(effects
@@
 		)
 	)
-	(label "IN30"
+	(label "IN2"
 		(at 193.04 43.18 180)
 		(effects
@@
 		)
 	)
-	(label "IN31"
+	(label "IN3"
 		(at 193.04 40.64 180)
 		(effects
@@
 		)
 	)
-	(label "IN29"
+	(label "IN1"
 		(at 224.79 41.91 180)
 		(effects
@@
 		)
 	)
-	(label "IN30"
+	(label "IN2"
 		(at 224.79 39.37 180)
 		(effects
@@
 		)
 	)
-	(label "IN28"
+	(label "IN0"
 		(at 256.54 41.91 180)
 		(effects
@@
 		)
 	)
-	(label "IN29"
+	(label "IN1"
 		(at 256.54 39.37 180)
 		(effects
@@
 		)
 	)
-	(label "IN34"
+	(label "IN6"
 		(at 226.06 82.55 180)
 		(effects
@@
 		)
 	)
-	(label "IN35"
+	(label "IN13"
 		(at 194.31 121.92 180)
 		(effects
@@
 		)
 	)
-	(label "IN36"
+	(label "IN14"
 		(at 130.81 125.73 180)
 		(effects
@@
 		)
 	)
-	(label "IN35"
+	(label "IN13"
 		(at 162.56 124.46 180)
 		(effects
@@
 		)
 	)
-	(label "IN37"
+	(label "IN15"
 		(at 130.81 123.19 180)
 		(effects
@@
 		)
 	)
-	(label "R1"
+	(label "R2"
 		(at 194.31 72.39 180)
 		(effects
@@
 		)
 	)
-	(label "IN37"
+	(label "IN9"
 		(at 130.81 83.82 180)
 		(effects
@@
 		)
 	)
-	(label "IN34"
+	(label "IN12"
 		(at 194.31 124.46 180)
 		(effects
@@
 		)
 	)
-	(label "IN37"
+	(label "C0"
+		(at 35.56 138.43 0)
+		(effects
+			(font
+				(size 1.27 1.27)
+			)
+			(justify left bottom)
+		)
+	)
+	(label "IN9"
 		(at 161.29 81.28 180)
 		(effects
@@
 		)
 	)
-	(label "R2"
+	(label "R4"
 		(at 130.81 115.57 180)
 		(effects
@@
 		)
 	)
-	(label "IN36"
+	(label "IN14"
 		(at 162.56 121.92 180)
 		(effects
@@
 		)
 	)
-	(label "R0"
+	(label "R2"
 		(at 194.31 114.3 180)
 		(effects
@@
 		)
 	)
-	(label "IN36"
+	(label "IN8"
 		(at 161.29 83.82 180)
 		(effects
@@
 		)
 	)
-	(label "R0"
+	(label "R1"
 		(at 226.06 72.39 180)
 		(effects
@@
 		)
 	)
-	(label "R3"
+	(label "R5"
 		(at 99.06 115.57 180)
 		(effects
@@
 		)
 	)
-	(label "IN37"
+	(label "IN15"
 		(at 99.06 125.73 180)
 		(effects
@@
 		)
 	)
-	(label "IN38"
+	(label "IN16"
 		(at 99.06 123.19 180)
 		(effects
@@
 		)
 	)
-	(label "IN35"
+	(label "IN7"
 		(at 226.06 80.01 180)
 		(effects
@@
 		)
 	)
-	(label "R1"
+	(label "R3"
 		(at 162.56 114.3 180)
 		(effects
@@
 		)
 	)
-	(label "IN40"
+	(label "IN12"
 		(at 226.06 123.19 180)
 		(effects
@@
 		)
 	)
-	(label "IN36"
+	(label "IN8"
 		(at 194.31 80.01 180)
 		(effects
@@
 		)
 	)
-	(label "IN38"
+	(label "IN10"
 		(at 257.81 125.73 180)
 		(effects
@@
 		)
 	)
-	(label "R2"
+	(label "R3"
 		(at 161.29 73.66 180)
 		(effects
@@
 		)
 	)
-	(label "R4"
+	(label "R0"
 		(at 257.81 115.57 180)
 		(effects
@@
 		)
 	)
-	(label "IN39"
+	(label "IN11"
 		(at 226.06 125.73 180)
 		(effects
@@
 		)
 	)
-	(label "IN39"
+	(label "IN11"
 		(at 257.81 123.19 180)
 		(effects
@@
 		)
 	)
-	(label "IN38"
+	(label "IN10"
 		(at 130.81 81.28 180)
 		(effects
@@
 		)
 	)
-	(label "R3"
+	(label "R4"
 		(at 130.81 73.66 180)
 		(effects
@@
 	)
 	(symbol
-		(lib_id "EasyEDA:HC-FPC-0.5-12P-FH20")
+		(lib_id "EasyEDA:HC-FPC-0.5-14P-FH20")
 		(at 43.18 121.92 0)
 		(unit 1)
@@
 			)
 		)
-		(property "Value" "HC-FPC-0.5-12P-FH20"
+		(property "Value" "HC-FPC-0.5-14P-FH20"
 			(at 50.8 123.1899 0)
 			(effects
@@
 			)
 		)
-		(property "Footprint" "EasyEDA:FPC-SMD_12P-P0.50_HC-FPC-0.5-12P-FH20"
+		(property "Footprint" "EasyEDA:FPC-SMD_14P-P0.50_HC-FPC-0.5-14P-FH20"
 			(at 43.18 148.59 0)
 			(effects
@@
 			)
 		)
-		(property "Datasheet" "https://www.lcsc.com/datasheet/C19273928.pdf"
+		(property "Datasheet" "https://www.lcsc.com/datasheet/C19273929.pdf"
 			(at 43.18 151.13 0)
 			(effects
@@
 			)
 		)
-		(property "MPN" "HC-FPC-0.5-12P-FH20"
+		(property "MPN" "HC-FPC-0.5-14P-FH20"
 			(at 43.18 156.21 0)
 			(effects
@@
 			)
 		)
-		(property "LCSC Part" "C19273928"
+		(property "LCSC Part" "C19273929"
 			(at 43.18 158.75 0)
 			(effects
@@
 		(pin "12"
 		)
+		(pin "16"
+		)
+		(pin "15"
+		)
+		(pin "13"
+		)
 		(pin "14"
 		)
-		(pin "13"
-		)
 		(instances
