File: 0.0.1-custom-pcb/rightPointerThumbBreakout/columnBreakout.kicad_pcb (KiCad board)
At the start: 2 copper layers, 28.7 x 63.3 mm, 17 parts, among them J1 HC-FPC-0.5-12P-FH20, J10 HC-FPC-0.5-6P-FH20, J11 HC-FPC-0.5-6P-FH20, J12 HC-FPC-0.5-6P-FH20, J13 HC-FPC-0.5-6P-FH20, J2 HC-FPC-0.5-6P-FH20, J3 HC-FPC-0.5-6P-FH20, J4 HC-FPC-0.5-6P-FH20, J5 HC-FPC-0.5-6P-FH20, J6 HC-FPC-0.5-6P-FH20, J7 HC-FPC-0.5-6P-FH20, J8 HC-FPC-0.5-6P-FH20, J9 HC-FPC-0.5-6P-FH20

Commit message: right pointerThumb before review
Parts:
- added J14: HC-FPC-0.5-6P-FH20, EasyEDA:FPC-SMD_6P-P0.50_HC-FPC-0.5-6P-FH20, F.Cu at (181.5, 90.7)
- added J15: HC-FPC-0.5-6P-FH20, EasyEDA:FPC-SMD_6P-P0.50_HC-FPC-0.5-6P-FH20, F.Cu at (181.5, 81.6)
- added J16: HC-FPC-0.5-6P-FH20, EasyEDA:FPC-SMD_6P-P0.50_HC-FPC-0.5-6P-FH20, F.Cu at (181.5, 72.5)
- added J17: HC-FPC-0.5-6P-FH20, EasyEDA:FPC-SMD_6P-P0.50_HC-FPC-0.5-6P-FH20, F.Cu at (181.5, 63.4)
- J1: value HC-FPC-0.5-12P-FH20 -> HC-FPC-0.5-14P-FH20; footprint EasyEDA:FPC-SMD_12P-P0.50_HC-FPC-0.5-12P-FH20 -> EasyEDA:FPC-SMD_14P-P0.50_HC-FPC-0.5-14P-FH20
- moved J13 38.9 mm to (181.5, 54.3)
- moved J12 38.9 mm to (181.5, 45.2)
- moved J1 21.4 mm to (175.4, 99.8)
- moved H2 13.8 mm to (186.7, 51.5)
- moved H4 13.8 mm to (186.7, 87.9)
- moved J9 9.10 mm to (167.8, 63.4)
- moved J8 9.10 mm to (167.8, 54.3)
- moved J11 8.90 mm to (167.8, 81.6)
- moved J10 8.80 mm to (167.8, 72.5)
Connections:
- net /IN28 renamed /IN0
- net /IN29 renamed /IN1
- net /IN30 renamed /IN2
- net /IN31 renamed /IN3
- net /IN32 renamed /IN4
- net /IN33 renamed /IN5
- net /IN34 renamed /IN6
- net /IN35 renamed /IN7
- net /IN36 renamed /IN8
- net /IN37 renamed /IN9
- net /IN38 renamed /IN10
- net /IN39 renamed /IN11
- J1 pad 11: /C6 -> /C2
- J1 pad 12: /C5 -> /C1
- J1 pad 13: unconnected-(J1-Pad13) -> /C0
- J1 pad 9: /IN40 -> /IN16
- J10 pad 1: /R2 -> /R3
- J10 pad 6: /C6 -> /C1
- J11 pad 1: /R3 -> /R4
- J11 pad 6: /C6 -> /C1
- J12 pad 1: /R4 -> /R0
- J12 pad 6: /C6 -> /C2
- J13 pad 1: /R5 -> /R1
- J13 pad 4: /IN40 -> /IN12
- J13 pad 6: /C6 -> /C2
- J2 pad 6: /C5 -> /C0
- J3 pad 6: /C5 -> /C0
- J4 pad 6: /C5 -> /C0
- J5 pad 6: /C5 -> /C0
- J6 pad 6: /C5 -> /C0
- J7 pad 6: /C5 -> /C0
- J8 pad 1: /R0 -> /R1
- J8 pad 6: /C6 -> /C1
- J9 pad 1: /R1 -> /R2
- J9 pad 6: /C6 -> /C1
Routing:
- net /GND: track 128.8 -> 256.7 mm, vias 13 -> 22
- net /VDD: track 129.8 -> 246.0 mm, vias 14 -> 22
- net /C0: track 0.00 -> 78.9 mm, vias 0 -> 2
- net /C6: track 65.2 -> 0.00 mm
- net /C2: track 0.00 -> 60.2 mm, vias 0 -> 2
- net /C5: track 55.3 -> 0.00 mm
- net /C1: track 0.00 -> 53.9 mm, vias 0 -> 2
- net /IN10: track 9.11 -> 57.1 mm, vias 0 -> 4
- net /R0: track 128.1 -> 83.3 mm, vias 4 -> 3
- net /R1: track 108.0 -> 75.3 mm
- net /R2: track 87.4 -> 66.2 mm
- net /IN0: track 55.4 -> 76.6 mm
- net /IN40: track 20.3 -> 0.00 mm, vias 2 -> 0
- net /IN16: track 0.00 -> 16.7 mm, vias 0 -> 2
- net /R3: track 68.3 -> 57.1 mm, vias 2 -> 4
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Other:
- board size 28.7 x 63.3 mm -> 42.5 x 63.3 mm
- board text added: "Col 0 →"
- board text added: "Col 1"
- board text added: "Col 2 →"
- board text added: "rightPointerThumbBreakout Rev 1"
- board text removed: "Col 5 →"
- board text removed: "Col 6 →"
- board text removed: "rightPinkieBreakout Rev 1"

Commit message: right pointerThumb ready for order
Routing:
- net /GND: track 256.7 -> 260.8 mm
- net /VDD: track 246.0 -> 248.4 mm
- net /IN10: track 57.1 -> 57.7 mm
