File: 0.0.1-custom-pcb/rightPinkieBreakout/routing-backups/before-highway-routing-20261006-214329.kicad_pcb (KiCad board)
At the start: 2 copper layers, 28.7 x 63.3 mm, 17 parts, among them J1 HC-FPC-0.5-12P-FH20, J10 HC-FPC-0.5-6P-FH20, J11 HC-FPC-0.5-6P-FH20, J12 HC-FPC-0.5-6P-FH20, J13 HC-FPC-0.5-6P-FH20, J2 HC-FPC-0.5-6P-FH20, J3 HC-FPC-0.5-6P-FH20, J4 HC-FPC-0.5-6P-FH20, J5 HC-FPC-0.5-6P-FH20, J6 HC-FPC-0.5-6P-FH20, J7 HC-FPC-0.5-6P-FH20, J8 HC-FPC-0.5-6P-FH20, J9 HC-FPC-0.5-6P-FH20

Commit message: left pinkie ready
Parts:
- moved J1 6.95 mm to (154.0, 99.8)
Routing:
- net /R0: track 69.5 -> 128.1 mm, vias 3 -> 4
- net /R1: track 60.4 -> 108.0 mm, vias 3 -> 4
- net /GND: track 166.6 -> 128.8 mm, vias 18 -> 13
- net /R2: track 51.0 -> 87.4 mm, vias 3 -> 4
- net /VDD: track 157.5 -> 129.8 mm, vias 18 -> 14
- net /R3: track 42.0 -> 68.3 mm, vias 3 -> 2
- net /R4: track 33.1 -> 48.5 mm, vias 3 -> 2
- net /IN34: track 66.8 -> 54.3 mm
- net /C5: track 63.9 -> 55.3 mm, vias 2 -> 0
- net /IN28: track 63.5 -> 55.4 mm
- net /IN40: track 13.7 -> 20.3 mm
- net /R5: track 24.0 -> 29.9 mm, vias 3 -> 2
- net /C6: track 59.7 -> 65.2 mm
- net /IN35: vias 0 -> 2
