File: 0.0.1-custom-pcb/rightPinkieBreakout/routing-backups/before-serial-move-20261006-222313.kicad_pcb (KiCad board)
At the start: 2 copper layers, 28.7 x 63.3 mm, 17 parts, among them J1 HC-FPC-0.5-12P-FH20, J10 HC-FPC-0.5-6P-FH20, J11 HC-FPC-0.5-6P-FH20, J12 HC-FPC-0.5-6P-FH20, J13 HC-FPC-0.5-6P-FH20, J2 HC-FPC-0.5-6P-FH20, J3 HC-FPC-0.5-6P-FH20, J4 HC-FPC-0.5-6P-FH20, J5 HC-FPC-0.5-6P-FH20, J6 HC-FPC-0.5-6P-FH20, J7 HC-FPC-0.5-6P-FH20, J8 HC-FPC-0.5-6P-FH20, J9 HC-FPC-0.5-6P-FH20

Commit message: left pinkie ready
Routing:
- net /C6: track 59.7 -> 62.2 mm
Changed lines of the file:
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@@
 	)
 	(gr_rect
-		(start 155.85 102.7)
-		(end 165.85 104.7)
+		(start 158.8 65)
+		(end 160.8 75)
 		(stroke
 			(width 0)
@@
 	)
 	(segment
+		(start 169 89.4)
+		(end 169 91.9)
+		(width 0.15)
+		(layer "F.Cu")
+		(net 14)
+	)
+	(segment
