File: 0.0.1-custom-pcb/leftPinkieBreakout/routing-backups/before-serial-reposition-20261006-224828.kicad_pcb (KiCad board)
At the start: 2 copper layers, 28.7 x 63.3 mm, 17 parts, among them J1 HC-FPC-0.5-12P-FH20, J10 HC-FPC-0.5-6P-FH20, J11 HC-FPC-0.5-6P-FH20, J12 HC-FPC-0.5-6P-FH20, J13 HC-FPC-0.5-6P-FH20, J2 HC-FPC-0.5-6P-FH20, J3 HC-FPC-0.5-6P-FH20, J4 HC-FPC-0.5-6P-FH20, J5 HC-FPC-0.5-6P-FH20, J6 HC-FPC-0.5-6P-FH20, J7 HC-FPC-0.5-6P-FH20, J8 HC-FPC-0.5-6P-FH20, J9 HC-FPC-0.5-6P-FH20

Commit message: all individual boards ready to print
Parts:
- moved J10 13.8 mm to (153.9, 63.7)
- moved J11 13.8 mm to (153.9, 72.7)
- moved J12 13.8 mm to (153.9, 81.6)
- moved J13 13.8 mm to (153.9, 90.7)
- moved J2 13.8 mm to (167.8, 45.2)
- moved J3 13.8 mm to (167.8, 54.3)
- moved J4 13.8 mm to (167.8, 63.4)
- moved J5 13.8 mm to (167.8, 72.5)
- moved J6 13.8 mm to (167.8, 81.6)
- moved J7 13.8 mm to (167.8, 90.7)
- moved J8 13.8 mm to (153.9, 45.2)
- moved J9 13.8 mm to (153.9, 54.3)
Routing:
- net /C5: track 63.9 -> 59.0 mm, vias 2 -> 0
- net /IN28: track 63.5 -> 60.0 mm
- net /C6: track 59.7 -> 62.6 mm, vias 0 -> 2
- net /IN40: track 13.7 -> 16.3 mm
- net /IN34: track 66.8 -> 65.4 mm
Other:
- board text added: "leftPinkieBreakout Rev 1"
- board text removed: "rightPinkieBreakout Rev 1"
