File: 0.0.1-custom-pcb/leftMainboard/leftMainboard.kicad_pcb (KiCad board)
At the start: 2 copper layers, 45 x 75 mm, 78 parts, among them J1 USB-C USB2 receptacle (footpr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, J10 HC-FPC-0.5-12P-FH20, J2 3-pin LiPo / NTC 1.25mm (esti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, J3 GPIO / SWD 2x6 1.27mm, J7 HC-FPC-0.5-14P-FH20, J8 HC-FPC-0.5-12P-FH20, J9 HC-FPC-0.5-12P-FH20, Q1 BSS138 (guess), Q2 P-channel MOSFET (guess), Q3 P-channel MOSFET (guess), SW1 Latching DPDT power push swit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, SW2 Reset tactile 4x4mm (estimate), U1 Boost controller MSOP8 (unide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, U2 TP4056-42-ESOP8, U3 PRTR5V0U2X, U4 MDBT50Q-P1MV2, U5 74CBTLV1G125GV (probable b25 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, Y1 32.768kHz (guess)

Commit message: left 12pin adjustment
Parts:
- moved J9 0.63 mm to (27.2, 55.6)
Routing:
- net IN22: track 13.5 -> 15.3 mm
