File: 0.0.1-custom-pcb/leftMainboard/Controller.kicad_sch (KiCad schematic)
At the start: 18 parts, among them J3 GPIO / SWD 2x6 1.27mm, Q1 BSS138 (guess), SW2 Reset tactile 4x4mm (estimate), U4 MDBT50Q-P1MV2, U5 74CBTLV1G125GV (probable b25 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, Y1 32.768kHz (guess)

Commit message: update more of left main
Parts:
- Q1: value BSS138 (guess) -> BSS138 N-channel; Confidence Low -> Medium; Evidence 3-lead packages; faint SS/G marking; polarity and part numb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 -> User measured body about 3x1.3 mm, marking SS; diode-mode d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; LCSC (none) -> C7420339
Changed lines of the file:
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@@
 (property "Reference" "Q1" (at 144.78 104.17999999999998 0)
 (effects (font (size 1.0 1.0))))
-(property "Value" "BSS138 (guess)" (at 144.78 114.25999999999999 0)
+(property "Value" "BSS138 N-channel" (at 144.78 114.25999999999999 0)
 (effects (font (size 0.8 0.8))))
 (property "Footprint" "Reconstruction:Q1_SOT-23" (at 144.78 109.21999999999998 0)
 (effects (font (size 1.0 1.0))
 (hide yes)))
-(property "Datasheet" "" (at 144.78 109.21999999999998 0)
+(property "Datasheet" "https://www.lcsc.com/datasheet/C7420339.pdf" (at 144.78 109.21999999999998 0)
 (effects (font (size 1.0 1.0))
 (hide yes)))
-(property "Confidence" "Low" (at 144.78 109.21999999999998 0)
+(property "LCSC" "C7420339" (at 144.78 109.21999999999998 0)
 (effects (font (size 1.0 1.0))
 (hide yes)))
-(property "Evidence" "3-lead packages; faint SS/G marking; polarity and part number unconfirmed" (at 144.78 109.21999999999998 0)
+(property "Confidence" "Medium" (at 144.78 109.21999999999998 0)
 (effects (font (size 1.0 1.0))
 (hide yes)))
+(property "Evidence" "User measured body about 3x1.3 mm, marking SS; diode-mode display 414 (about 0.414 V), pins 1/2 shorted, red 2 black 3; supports N-channel; reverse reading and isolated-device test not reported; exact MPN unconfirmed" (at 144.78 109.21999999999998 0)
+(effects (font (size 1.0 1.0))
+(hide yes)))

Commit message: more left main updates2
Parts:
- SW2: value Reset tactile 4x4mm (estimate) -> TS3735A 250gf 030; footprint Reconstruction:Reset_Tactile_4mm_PhotoEstimate -> Reconstruction:SW_TS3735A_C2906282_EasyEDA; symbol Reconstruction:SW2_Reset_Tactile_4mm_PhotoEstimate -> Reconstruction:SW2_TS3735A_C2906282; Candidate part 4x4mm SMT tactile switch -> C2906282 / TS3735A 250gf 030; Confidence Medium -> User-selected replacement; original part unconfirmed; Evidence Yellow tactile dome in photo beside module -> User-selected C2906282; footprint and 3D models imported fr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; LCSC (none) -> C2906282; LCSC Part (none) -> C2906282; MPN (none) -> TS3735A 250gf 030; Manufacturer (none) -> SHOU HAN
Connections:
- net GND: now also SW2.3, SW2.4; no longer SW2.2
- net RESET: now also SW2.2
Changed lines of the file:
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@@
 (effects (font (size 1.0 1.0))
 (hide yes))))
-(symbol (lib_id "Reconstruction:SW2_Reset_Tactile_4mm_PhotoEstimate")
-(at 144.78 231.13999999999993 0)
-(unit 1)
-(exclude_from_sim no)
-(in_bom yes)
-(on_board yes)
-(dnp no)
-(property "Reference" "SW2" (at 144.78 226.09999999999994 0)
-(effects (font (size 1.0 1.0))))
-(property "Value" "Reset tactile 4x4mm (estimate)" (at 144.78 236.17999999999992 0)
-(effects (font (size 0.8 0.8))))
-(property "Footprint" "Reconstruction:Reset_Tactile_4mm_PhotoEstimate" (at 144.78 231.13999999999993 0)
-(effects (font (size 1.0 1.0))
-(hide yes)))
-(property "Datasheet" "" (at 144.78 231.13999999999993 0)
-(effects (font (size 1.0 1.0))
-(hide yes)))
-(property "Confidence" "Medium" (at 144.78 231.13999999999993 0)
-(effects (font (size 1.0 1.0))
-(hide yes)))
-(property "Evidence" "Yellow tactile dome in photo beside module" (at 144.78 231.13999999999993 0)
-(effects (font (size 1.0 1.0))
-(hide yes)))
-(property "Candidate part" "4x4mm SMT tactile switch" (at 144.78 231.13999999999993 0)
-(effects (font (size 1.0 1.0))
-(hide yes)))
-(pin "1")
-(pin "2")
-(instances (project "leftMainboard" (path "/eac6e0a1-0901-4c4d-b0b4-c941afc6d33b/2e843c11-c64d-453b-b36a-ba1514fd61ab" (reference "SW2")
-(unit 1)))))
+(symbol (lib_id "Reconstruction:SW2_TS3735A_C2906282") (at 144.78 231.13999999999993 0) (unit 1) (exclude_from_sim no) (in_bom yes) (on_board yes) (dnp no) (property "Reference" "SW2" (at 144.78 226.09999999999994 0) (effects (font (size 1.0 1.0)))) (property "Value" "TS3735A 250gf 030" (at 144.78 236.17999999999992 0) (effects (font (size 0.8 0.8)))) (property "Footprint" "Reconstruction:SW_TS3735A_C2906282_EasyEDA" (at 144.78 231.13999999999993 0) (effects (font (size 1.0 1.0)) (hide yes))) (property "Datasheet" "https://www.lcsc.com/datasheet/C2906282.pdf" (at 144.78 231.13999999999993 0) (effects (font (size 1.0 1.0)) (hide yes))) (property "Confidence" "User-selected replacement; original part unconfirmed" (at 144.78 231.13999999999993 0) (effects (font (size 1.0 1.0)) (hide yes))) (property "Evidence" "User-selected C2906282; footprint and 3D models imported from JLCEDA/EasyEDA Official Library; common pin pairs 1/2 and 3/4 checked against manufacturer drawing" (at 144.78 231.13999999999993 0) (effects (font (size 1.0 1.0)) (hide yes))) (property "Candidate part" "C2906282 / TS3735A 250gf 030" (at 144.78 231.13999999999993 0) (effects (font (size 1.0 1.0)) (hide yes))) (pin "1") (pin "3") (instances (project "leftMainboard" (path "/eac6e0a1-0901-4c4d-b0b4-c941afc6d33b/2e843c11-c64d-453b-b36a-ba1514fd61ab" (reference "SW2") (unit 1)))) (property "Description" "SHOU HAN 3.7x3.7mm low-profile momentary tactile switch, 250gf" (at 144.78 231.13999999999993 0) (effects (font (size 1.0 1.0)) (hide yes))) (property "Manufacturer" "SHOU HAN" (at 144.78 231.13999999999993 0) (effects (font (size 1.0 1.0)) (hide yes))) (property "MPN" "TS3735A 250gf 030" (at 144.78 231.13999999999993 0) (effects (font (size 1.0 1.0)) (hide yes))) (property "LCSC" "C2906282" (at 144.78 231.13999999999993 0) (effects (font (size 1.0 1.0)) (hide yes))) (property "LCSC Part" "C2906282" (at 144.78 231.13999999999993 0) (effects (font (size 1.0 1.0)) (hide yes))) (pin "2") (pin "4"))
 (wire (pts (xy 223.52 46.99)
 (xy 218.44 46.99))
@@
 (effects (font (size 1.0 1.0))
 (justify left))
-))
+)(wire (pts (xy 134.62 229.87) (xy 134.62 232.41)) (stroke (width 0) (type default)))
+(wire (pts (xy 154.94 229.87) (xy 154.94 232.41)) (stroke (width 0) (type default)))
+)
