File: 0.0.1-custom-pcb/leftMainboard/PowerAndUSB.kicad_sch (KiCad schematic)
At the start: 31 parts, among them J1 USB-C USB2 receptacle (footpr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, J2 53398-0371, Q2 P-channel MOSFET (guess), Q3 BSS138 N-channel, SW1 TK-6580A-1, U1 SY7088DGC, U2 TP4056-42-ESOP8, U3 PRTR5V0U2X

Commit message: more left main updates2
Parts:
- Q2: value P-channel MOSFET (guess) -> DMG2305UX; Candidate part AO3401A / SI2301 family -> C2940629 / DMG2305UX; Confidence Low -> User-selected replacement; P-channel confirmed by user; Evidence 3-lead packages; faint SS/G marking; polarity and part numb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 -> User confirmed P-channel by multimeter; reported 5PEY marki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; LCSC (none) -> C2940629; LCSC Part (none) -> C2940629; MPN (none) -> DMG2305UX; Manufacturer (none) -> TECH PUBLIC
Connections:
- net VBAT: no longer SW1.1 (COM_A)
- net VBAT_SWITCHED renamed SW1_ON_VDDH
- net SW1_ON_VDDH: no longer SW1.6 (NO_B)
- new net SW1_OFF_VBAT: SW1.1 (COM_A)
- no-connect marks 4 -> 5
Changed lines of the file:
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@@
 (type default))
 )
-(global_label "VBAT" (shape passive)
+(global_label "SW1_OFF_VBAT" (shape passive)
 (at 40.64 105.41 0)
 (effects (font (size 0.9 0.9)))
@@
 (type default))
 )
-(global_label "VBAT_SWITCHED" (shape passive)
+(global_label "SW1_ON_VDDH" (shape passive)
 (at 40.64 107.95 0)
 (effects (font (size 0.9 0.9)))
@@
 (effects (font (size 0.9 0.9)))
 (property "Intersheetrefs" "${INTERSHEET_REFS}" (at 71.12 105.41 0)
-(effects (font (size 1.0 1.0))
-(hide yes))))
-(wire (pts (xy 66.04 107.95)
-(xy 71.12 107.95))
-(stroke (width 0)
-(type default))
-)
-(global_label "VBAT_SWITCHED" (shape passive)
-(at 71.12 107.95 180)
-(effects (font (size 0.9 0.9)))
-(property "Intersheetrefs" "${INTERSHEET_REFS}" (at 71.12 107.95 0)
 (effects (font (size 1.0 1.0))
 (hide yes))))
@@
 (type default))
 )
-(global_label "VBAT_SWITCHED" (shape passive)
+(global_label "SW1_ON_VDDH" (shape passive)
 (at 40.64 204.47 0)
 (effects (font (size 0.9 0.9)))
@@
 (property "Reference" "Q2" (at 55.88 198.15999999999997 0)
 (effects (font (size 1.0 1.0))))
-(property "Value" "P-channel MOSFET (guess)" (at 55.88 208.23999999999995 0)
+(property "Value" "DMG2305UX" (at 55.88 208.23999999999995 0)
 (effects (font (size 0.8 0.8))))
 (property "Footprint" "Reconstruction:Q2_SOT-23" (at 55.88 203.19999999999996 0)
 (effects (font (size 1.0 1.0))
 (hide yes)))
-(property "Datasheet" "" (at 55.88 203.19999999999996 0)
-(effects (font (size 1.0 1.0))
-(hide yes)))
-(property "Confidence" "Low" (at 55.88 203.19999999999996 0)
-(effects (font (size 1.0 1.0))
-(hide yes)))
-(property "Evidence" "3-lead packages; faint SS/G marking; polarity and part number unconfirmed" (at 55.88 203.19999999999996 0)
-(effects (font (size 1.0 1.0))
-(hide yes)))
-(property "Candidate part" "AO3401A / SI2301 family" (at 55.88 203.19999999999996 0)
+(property "Datasheet" "https://www.lcsc.com/datasheet/C2940629.pdf" (at 55.88 203.19999999999996 0)
+(effects (font (size 1.0 1.0))
+(hide yes)))
+(property "Confidence" "User-selected replacement; P-channel confirmed by user" (at 55.88 203.19999999999996 0)
+(effects (font (size 1.0 1.0))
+(hide yes)))
+(property "Evidence" "User confirmed P-channel by multimeter; reported 5PEY marking matches manufacturer 5Pxx marking format; user-selected C2940629" (at 55.88 203.19999999999996 0)
+(effects (font (size 1.0 1.0))
+(hide yes)))
+(property "Candidate part" "C2940629 / DMG2305UX" (at 55.88 203.19999999999996 0)
 (effects (font (size 1.0 1.0))
 (hide yes)))
@@
 (pin "3")
 (instances (project "leftMainboard" (path "/eac6e0a1-0901-4c4d-b0b4-c941afc6d33b/3d4a4145-dfbf-4d53-839d-da2f670b524e" (reference "Q2")
-(unit 1)))))
+(unit 1))))
+(property "Description" "TECH PUBLIC DMG2305UX P-channel MOSFET, SOT-23, selected replacement C2940629" (at 55.88 203.19999999999996 0)
+(effects (font (size 1.0 1.0))
+(hide yes)))
+(property "Manufacturer" "TECH PUBLIC" (at 55.88 203.19999999999996 0)
+(effects (font (size 1.0 1.0))
+(hide yes)))
+(property "MPN" "DMG2305UX" (at 55.88 203.19999999999996 0)
+(effects (font (size 1.0 1.0))
+(hide yes)))
+(property "LCSC" "C2940629" (at 55.88 203.19999999999996 0)
+(effects (font (size 1.0 1.0))
+(hide yes)))
+(property "LCSC Part" "C2940629" (at 55.88 203.19999999999996 0)
+(effects (font (size 1.0 1.0))
+(hide yes)))
+)
 (wire (pts (xy 45.72 222.25)
 (xy 40.64 222.25))
@@
 (symbol (lib_id "Reconstruction:ExternalPowerFlag") (at 88.9 127.0 0) (unit 1) (exclude_from_sim no) (in_bom no) (on_board yes) (dnp no) (property "Reference" "#FLG0102" (at 88.9 125.095 0) (effects (font (size 1.27 1.27)) (hide yes))) (property "Value" "PWR_FLAG" (at 88.9 123.19 0) (effects (font (size 1.27 1.27)))) (property "Footprint" "" (at 88.9 127.0 0) (effects (font (size 1.27 1.27)) (hide yes))) (property "Datasheet" "~" (at 88.9 127.0 0) (effects (font (size 1.27 1.27)) (hide yes))) (property "Description" "Special symbol for telling ERC where power comes from" (at 88.9 127.0 0) (effects (font (size 1.27 1.27)) (hide yes))) (property "ki_keywords" "flag power" (at 88.9 127.0 0) (effects (font (size 1.27 1.27)) (hide yes))) (pin "1") (instances (project "leftMainboard" (path "/eac6e0a1-0901-4c4d-b0b4-c941afc6d33b/3d4a4145-dfbf-4d53-839d-da2f670b524e" (reference "#FLG0102") (unit 1)))))
 (global_label "VDDH" (shape passive) (at 88.9 127.0 0) (effects (font (size 0.9 0.9))) (property "Intersheetrefs" "${INTERSHEET_REFS}" (at 88.9 127.0 0) (effects (font (size 1.0 1.0)) (hide yes))))
-)
+	(no_connect (at 66.04 107.95))
+)
